File: rf2/head/out/SB1R_RF2/SB1R-QA-RF2.kicad_pcb (KiCad board)
At the start: 4 copper layers, 228 x 228 mm, 9 parts

Commit message: WIP snapshot: electrician (NTBG / clamp / cord) and draftsman (bank winding, PRX, QA/QB, glove housing) agents in progress
Co-Authored-By: Claude Opus 5.5 <noreply@anthropic.com>
Claude-Session: https://claude.ai/code/session_01JecXWNPV9NmFDovQZQG27P
Parts:
- added H4: , SB1R:MH_M3, F.Cu at (99.1, 69.1)
Changed lines of the file:
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@@
   (footprint "SB1R:MH_M3" (layer "F.Cu") (at 124.131 109.285) (property "Reference" "H2" (at 0 -3) (layer "F.SilkS")) (pad "" np_thru_hole circle (at 0 0) (size 3.4 3.4) (drill 3.4) (layers "*.Cu" "*.Mask")))
   (footprint "SB1R:MH_M3" (layer "F.Cu") (at 139.285 145.869) (property "Reference" "H3" (at 0 -3) (layer "F.SilkS")) (pad "" np_thru_hole circle (at 0 0) (size 3.4 3.4) (drill 3.4) (layers "*.Cu" "*.Mask")))
+  (footprint "SB1R:MH_M3" (layer "F.Cu") (at 99.088 69.088) (property "Reference" "H4" (at 0 -3) (layer "F.SilkS")) (pad "" np_thru_hole circle (at 0 0) (size 3.4 3.4) (drill 3.4) (layers "*.Cu" "*.Mask")))
   (segment (start 177.0569 102.7661) (end 179.9562 104.6157) (width 0.8) (layer "F.Cu") (net 1))
   (segment (start 179.9562 104.6157) (end 183.0036 106.2094) (width 0.8) (layer "F.Cu") (net 1))
